File: IntroBoard/untitled.kicad_sch (KiCad schematic)
At the start: 23 parts, among them J1 3220-20-0200-00, J2 USB PLUG, J3 647676-2, J4 1984617, U3 ${SIM.PARAMS}, U7 USB CHIP

Commit message: 1.1
Quick fixes after review
Parts:
- R5: value 10k -> 1k
Connections:
- net GND: now also U7.21 (EPAD)
- no-connect marks 23 -> 22
Changed lines of the file:
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@@
 	)
 	(no_connect
-		(at 101.6 67.31)
-	)
-	(no_connect
 		(at 123.19 45.72)
 	)
@@
 	(wire
 		(pts
+			(xy 96.52 67.31) (xy 96.52 68.58)
+		)
+		(stroke
+			(width 0)
+			(type default)
+		)
+	)
+	(wire
+		(pts
 			(xy 30.48 60.96) (xy 30.48 63.5)
 		)
@@
 	(wire
 		(pts
+			(xy 101.6 67.31) (xy 96.52 67.31)
+		)
+		(stroke
+			(width 0)
+			(type default)
+		)
+	)
+	(wire
+		(pts
 			(xy 140.97 97.79) (xy 167.64 97.79)
 		)
@@
 	)
 	(symbol
+		(lib_id "power:GND")
+		(at 96.52 68.58 0)
+		(unit 1)
+		(exclude_from_sim no)
+		(in_bom yes)
+		(on_board yes)
+		(dnp no)
+		(property "Reference" "#PWR023"
+			(at 96.52 74.93 0)
+			(effects
+				(font
+					(size 1.27 1.27)
+				)
+				(hide yes)
+			)
+		)
+		(property "Value" "GND"
+			(at 92.71 71.12 0)
+			(effects
+				(font
+					(size 1.27 1.27)
+				)
+			)
+		)
+		(property "Footprint" ""
+			(at 96.52 68.58 0)
+			(effects
+				(font
+					(size 1.27 1.27)
+				)
+				(hide yes)
+			)
+		)
+		(property "Datasheet" ""
+			(at 96.52 68.58 0)
+			(effects
+				(font
+					(size 1.27 1.27)
+				)
+				(hide yes)
+			)
+		)
+		(property "Description" "Power symbol creates a global label with name \"GND\" , ground"
+			(at 96.52 68.58 0)
+			(effects
+				(font
+					(size 1.27 1.27)
+				)
+				(hide yes)
+			)
+		)
+		(pin "1"
+		)
+		(instances
+			(project ""
+				(path "/8b361d18-084e-4f41-9927-72e4c0f07c3e/3ec74b54-7181-4525-b4fc-3d9e1217fe1f"
+					(reference "#PWR023")
+					(unit 1)
+				)
+			)
+		)
+	)
+	(symbol
 		(lib_id "Device:C")
 		(at 172.72 86.36 0)
@@
 			)
 		)
-		(property "Value" "10k"
+		(property "Value" "1k"
 			(at 143.51 74.93 0)
 			(effects

Commit message: 1.2
Quickfix
Parts:
- added Q1: NMOS, Coolstuff:SOT95P240X111-3N, symbol Simulation_SPICE:NMOS
- added R18: 10k, Resistor_SMD:R_0603_1608Metric, symbol Device:R
- R5: value 1k -> 10k
Connections:
- net 3.3V: now also LS1.P, R18.1
- net BUZZ: now also Q1.2 (G); no longer LS1.P
- net GND: now also Q1.3 (S); no longer LS1.N
- net at U7.13 (WAKEUP): now also R18.2
- net GPIO_OUT4 renamed BRIDGE_RSTB
- net USART2_RX renamed BRIDGE_RX
- net USART2_TX renamed BRIDGE_TX
- new net: LS1.N, Q1.1 (D)
- no-connect marks 22 -> 21
Other:
- note removed: "continuity switch terminal to power lipo review uart bridge control LED (program)"
- moved on the sheet: D2, LS1, R15
