File: IntroBoard/IntroBoard.kicad_pcb (KiCad board)
At the start: 4 copper layers, 81.5 x 34.5 mm, 53 parts, among them J1 3220-20-0200-00, J2 USB PLUG, J3 647676-2, J4 1984617, SW1 SW_SPST, U1 FLASH, U2 STM32G441KBT6, U4 BMI323, U5 LMS8117AMP-3.3/NOPB, U6 BMP390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

Commit message: 1.2
Quickfix
Parts:
- removed SW1: SW_SPST, Button_Switch_SMD:SW_SPST_PTS647_Sx38
- added C16: 1uF, Capacitor_SMD:C_0603_1608Metric, F.Cu at (125.5, 103.0)
- added C8: 4.7uF, Capacitor_SMD:C_0603_1608Metric, F.Cu at (110.8, 111.0)
- added JP2: Jumper_2_Open, TestPoint:TestPoint_2Pads_Pitch2.54mm_Drill0.8mm, F.Cu at (102.5, 111.2)
- added Q1: NMOS, Coolstuff:SOT95P240X111-3N, F.Cu at (93.5, 109.4)
- added R16: 10k, Resistor_SMD:R_0603_1608Metric, F.Cu at (119.5, 97.5)
- added R17: 10k, Resistor_SMD:R_0603_1608Metric, F.Cu at (121.5, 94.0)
- added R18: 10k, Resistor_SMD:R_0603_1608Metric, F.Cu at (136.5, 105.8)
- C3, C5: value 0.1uF -> 100nF
- C6: value 0.1 nF -> 0.1 uF
- C7: value 0.1uF -> 10nF
- moved C2 0.10 mm to (112.8, 113.5)
Connections:
- net EXTI11 renamed IMU_INT1
- net EXTI12 renamed IMU_INT2
- net EXTI6 renamed BARO_INT
- net GPIO_OUT1 renamed FLASH_CE
- net GPIO_OUT2 renamed FLASH_HOLD
- net GPIO_OUT3 renamed FLASH_WP
- net GPIO_OUT4 renamed BRIDGE_RSTB
- net I2C1_SCK renamed BARO_SCK
- net I2C1_SDA renamed BARO_SDA
- net I2C2_SCK renamed IMU_SCK
- net I2C2_SDA renamed IMU_SDA
- net SPI1_MISO renamed FLASH_MISO
- net SPI1_MOSI renamed FLASH_MOSI
- net SPI1_SCK renamed FLASH_SCK
- net USART2_RX renamed BRIDGE_RX
- net USART2_TX renamed BRIDGE_TX
- LS1 pad N: GND -> Net-(Q1-D)
- LS1 pad P: BUZZ -> 3.3V
- U4 pad 1: unconnected-(U4-SDO-Pad1) -> GND
- U7 pad 13: unconnected-(U7-WAKEUP-Pad13) -> Net-(U7-WAKEUP)
- U7 pad 21: unconnected-(U7-EPAD-Pad21) -> GND
Routing:
- net 3.3V: track 75.2 -> 87.7 mm
- net Net-(Q1-D): track 0.00 -> 10.5 mm
- net BUZZ: track 17.5 -> 26.1 mm, vias 2 -> 4
- net NRST: track 39.5 -> 35.7 mm
- net IMU_SCK: track 11.3 -> 14.7 mm
- net GND: track 112.2 -> 115.0 mm, vias 24 -> 28
- net IMU_SDA: track 9.54 -> 12.3 mm
- net Net-(U7-WAKEUP): track 0.00 -> 1.91 mm
- net SWDIO: track 13.5 -> 14.4 mm
- net BRIDGE_TX: track 24.3 -> 24.9 mm
- net BRIDGE_RX: track 21.6 -> 22.1 mm

Commit message: Final Touches
Finished (theoretically) intro board
Parts:
- removed C2, C4: 7pF, Capacitor_SMD:C_0603_1608Metric
- removed X1: 32.768kHz, Coolstuff:XTAL_CM7V-T1A_MCX
- added LOGO1: Logo, Flight-Computer:Logo, F.Cu at (94.5, 86.5)
- added Y1: ECS-327TXO-33-TR, Coolstuff:OSC_ECS-327TXO-33-TR, F.Cu at (115.4, 112.8)
- C5: value 100nF -> 10nF
- C7: value 10nF -> 100nF
- CR2, CR3: value SM5819PL-TP -> MSS1P3L-M3/89A; footprint Coolstuff:SOD-123FL_MCC -> Diode_SMD:D_MicroSMP_AK
- U5: value LMS8117AMP-3.3/NOPB -> MIC5501-3.0YM5-TR; footprint Coolstuff:LINREG -> Coolstuff:SOT23-5LD-PL-1_MCH
- moved R15 2.50 mm to (99.2, 92.5)
- moved U5 1.80 mm to (142.0, 88.0), turned to 90 degrees
- moved D2 1.50 mm to (103.5, 91.5)
Connections:
- U2 pad 3: OSC_OUT -> unconnected-(U2-PF1-OSC_OUT-Pad3)
- U5 pad 1: GND -> VIN
- U5 pad 2: 3.3V -> GND
Routing:
- net 3.3V: track 87.7 -> 98.4 mm, vias 15 -> 18
- net OSC_OUT: track 5.54 -> 0.00 mm
- net GND: track 115.0 -> 119.3 mm
- net VIN: track 36.6 -> 40.7 mm
- net OSC_IN: track 5.13 -> 2.93 mm
- net LIGHTS: track 19.4 -> 17.9 mm
