File: IntroBoard/IntroBoard.kicad_sch (KiCad schematic)
At the start: 30 parts, among them SW1 SW_SPST, U1 FLASH, U2 STM32G441KBT6, U4 BMI323, U5 LMS8117AMP-3.3/NOPB, U6 BMP390, X1 32.768kHz

Commit message: 1.1
Quick fixes after review
Parts:
- added C16, C8: 100nF, Capacitor_SMD:C_0603_1608Metric, symbol Device:C
- added R16: R, symbol Device:R
- added R17: 10k, symbol Device:R
- C3, C7: value 0.1uF -> 100nF
- C5: value 0.1uF -> 10nF
Connections:
- net 3.3V: now also C16.1, C8.1, R17.2; no longer U6.6 (CSB)
- net GND: now also C16.2, C8.2, R16.1
- net at U4.1 (SDO): now also R16.2
- new net: R17.1, U6.6 (CSB)
- no-connect marks 1 -> 0
Other:
- note added: "CHANGED"
- moved on the sheet: C3, C5, C7

Commit message: 1.2
Quickfix
Parts:
- removed SW1: SW_SPST, Button_Switch_SMD:SW_SPST_PTS647_Sx38, symbol Switch:SW_SPST
- added JP2: Jumper_2_Open, TestPoint:TestPoint_2Pads_Pitch2.54mm_Drill0.8mm, symbol Jumper:Jumper_2_Open
- C16: value 100nF -> 1uF
- C6: value 0.1 nF -> 0.1 uF
- C8: value 100nF -> 4.7uF
- R16: value R -> 10k; footprint (none) -> Resistor_SMD:R_0603_1608Metric
- R17: footprint (none) -> Resistor_SMD:R_0603_1608Metric
Connections:
- net I2C2_SCK is gone; now on net IMU_SCK: U2.19 (PA9), U4.13 (SCX)
- net I2C2_SDA is gone; now on net IMU_SDA: U2.18 (PA8), U4.14 (SDX)
- net 3.3V: now also R16.1, U6.6 (CSB)
- net GND: now also U4.1 (SDO), JP2.2 (B); no longer R16.1
- net NRST: now also JP2.1 (A)
- net IMU_SDA: now reaches R16.2
- net IMU_SDA: no longer U4.1 (SDO)
- net IMU_SCK: now reaches R17.1
- net IMU_SCK: no longer U6.6 (CSB)
- net EXTI11 renamed IMU_INT1
- net EXTI12 renamed IMU_INT2
- net EXTI6 renamed BARO_INT
- net GPIO_OUT1 renamed FLASH_CE
- net GPIO_OUT2 renamed FLASH_HOLD
- net GPIO_OUT3 renamed FLASH_WP
- net GPIO_OUT4 renamed BRIDGE_RSTB
- net I2C1_SCK renamed BARO_SCK
- net I2C1_SDA renamed BARO_SDA
- net SPI1_MISO renamed FLASH_MISO
- net SPI1_MOSI renamed FLASH_MOSI
- net SPI1_SCK renamed FLASH_SCK
- net USART2_RX renamed BRIDGE_RX
- net USART2_TX renamed BRIDGE_TX
Other:
- note added: "0x69"
- note added: "0x77"
- note added: "REMIND TO INITALIZE ALL PINS"
- note removed: "continuity switch terminal to power lipo review uart bridge control LED (program)"
- note removed: "tant caps"
- moved on the sheet: C1, C11, C13, C3, C5, C7, C9, U1, U4

Commit message: Final Touches
Finished (theoretically) intro board
Parts:
- removed C2, C4: 7pF, Capacitor_SMD:C_0603_1608Metric, symbol Device:C
- removed U5: LMS8117AMP-3.3/NOPB, Coolstuff:LINREG, symbol LINREG:LMS8117AMP-3.3_NOPB
- removed X1: 32.768kHz, Coolstuff:XTAL_CM7V-T1A_MCX, symbol CRYSTRES:CM7V-T1A-32.768KHZ-7PF-20PPM-TA-QC
- added U5: MIC5501-3.0YM5-TR, Coolstuff:SOT23-5LD-PL-1_MCH, symbol LINREG:MIC5501-3.0YM5-TR
- added Y1: ECS-327TXO-33-TR, Coolstuff:OSC_ECS-327TXO-33-TR, symbol CRYSTRES:ECS-327TXO-33-TR
- CR2, CR3: value SM5819PL-TP -> MSS1P3L-M3/89A; footprint Coolstuff:SOD-123FL_MCC -> Diode_SMD:D_MicroSMP_AK
Connections:
- net 3.3V: now also U5.5 (VOUT), Y1.1 (OE), Y1.4 (SUPPLY_VOLTAGE)
- net GND: now also U5.2 (GND), Y1.2 (GND)
- net OSC_IN: now also Y1.3 (OUTPUT)
- net VIN: now also U5.1 (VIN), U5.3 (EN)
- net OSC_OUT: no longer names the net of U2.3 (PF1-OSC_OUT)
- no-connect marks 0 -> 1
Other:
- note removed: "CHANGED"
- moved on the sheet: C6, JP2
